File: POLOLUS_AXIS.sch (KiCad schematic (older format))
At the start: 0 parts

Commit message: Adicion de documentacion
Creacion y adicion de componente A4988 en hoja POLOLUS_AXIS.sch, Avance parcialmente completo de  hoja POLOLUS_AXIS.sch
Parts:
- added C? (x3): CP, symbol CP
- added P? (x6): CONN_01X03, symbol CONN_01X03
- added P? (x3): CONN_01X04, symbol CONN_01X04
- added P?: CONN_01X02, symbol CONN_01X02
- added U? (x3): A4988, symbol A4988
Connections:
- new net: P?.1 (P1), U?.10 (MS1) (x3)
- new net: P?.2 (P2), U?.11 (MS2) (x3)
- new net: P?.3 (P3), U?.12 (MS3) (x3)
- new net: U?.13 (RST), U?.14 (SLP) (x3)
- new net: P?.1 (P1), U?.3 (1B) (x3)
- new net: P?.2 (P2), U?.4 (1A) (x3)
- new net: P?.3 (P3), U?.5 (2A) (x3)
- new net: P?.4 (P4), U?.6 (2B) (x3)
- new net: C?.1, C?.1, C?.1, P?.1 (P1), U?.8 (VMOT), U?.8 (VMOT), U?.8 (VMOT)
- new net +5V: P?.1 (P1), P?.1 (P1), P?.1 (P1), P?.2 (P2), P?.2 (P2), P?.2 (P2), P?.3 (P3), P?.3 (P3), P?.3 (P3), U?.2 (VDD), U?.2 (VDD), U?.2 (VDD)
- new net DIR1: U?.16 (DIR)
- new net DIR2: U?.16 (DIR)
- new net DIR3: U?.16 (DIR)
- new net ENABLE: U?.9 (ENA), U?.9 (ENA), U?.9 (ENA)
- new net GND: C?.2, C?.2, C?.2, P?.2 (P2), U?.1 (GND), U?.1 (GND), U?.1 (GND), U?.7 (GND), U?.7 (GND), U?.7 (GND)
- new net STEP1: U?.15 (STEP)
- new net STEP2: U?.15 (STEP)
- new net STEP3: U?.15 (STEP)

Commit message: Reorganizacion de carpetas y avance de esquematico
Creacion de componente LM2596. Hoja REGULADOR finalizada. Avance parcial en hoja CONECTOR_EDU_CIAA. Creacion de carpetas datasheet y doc. Adicion de hojas de datos de LM2596, A4988, MMBT2222A. Adicion de documentacion LICENCIA, README, Revisiones.
Parts:
- removed P?: CONN_01X02, symbol CONN_01X02
- gave numbers to parts that had none: 15
Connections:
- net +5V: no longer U2.2 (VDD), U3.2 (VDD), U4.2 (VDD)
- net EXT-V: now reaches C3.1, C4.1, C5.1, U2.8 (VMOT), U3.8 (VMOT), U4.8 (VMOT)
- new net +3V3: U2.2 (VDD), U3.2 (VDD), U4.2 (VDD)
Changed lines of the file:
@@
 encoding utf-8
 Sheet 4 4
-Title ""
+Title "CNC Poncho - Controladores de Motore Paso a Paso"
 Date "2016-11-26"
 Rev "1.0"
 Comp "CESE - Curso de diseño de PCB"
 Comment1 "Autor: Marcelo Franz Moreno Marin"
-Comment2 "Licencia:"
+Comment2 "Licencia: doc/LICENCIA"
 Comment3 ""
 Comment4 ""
 $EndDescr
 $Comp
-L A4988 U?
+L A4988 U2
 U 1 1 583A501D
 P 4050 2150
-F 0 "U?" H 4050 2600 60  0000 C CNN
+F 0 "U2" H 4050 2600 60  0000 C CNN
 F 1 "A4988" H 4050 1700 60  0000 C CNN
 F 2 "" H 3950 2350 60  0001 C CNN
@@
 $EndComp
 $Comp
-L A4988 U?
+L A4988 U3
 U 1 1 583A52A2
 P 4050 3650
-F 0 "U?" H 4050 4100 60  0000 C CNN
+F 0 "U3" H 4050 4100 60  0000 C CNN
 F 1 "A4988" H 4050 3200 60  0000 C CNN
 F 2 "" H 3950 3850 60  0001 C CNN
@@
 $EndComp
 $Comp
-L A4988 U?
+L A4988 U4
 U 1 1 583A52EC
 P 4050 5150
-F 0 "U?" H 4050 5600 60  0000 C CNN
+F 0 "U4" H 4050 5600 60  0000 C CNN
 F 1 "A4988" H 4050 4700 60  0000 C CNN
 F 2 "" H 3950 5350 60  0001 C CNN
@@
 	2200 4800 3550 4800
 Wire Wire Line
-	4550 5500 6300 5500
-Wire Wire Line
 	4550 4900 4900 4900
 Wire Wire Line
 	4900 4900 4900 5650
 Wire Wire Line
-	4550 4000 5700 4000
-Wire Wire Line
-	4550 2500 5700 2500
-Wire Wire Line
 	4550 3400 4900 3400
 Wire Wire Line
@@
 	4900 1900 4900 2650
 $Comp
-L CONN_01X03 P?
+L CONN_01X03 P11
 U 1 1 583A5FE7
 P 3200 2000
-F 0 "P?" H 3200 1800 50  0000 C CNN
+F 0 "P11" H 3200 1800 50  0000 C CNN
 F 1 "CONN_01X03" V 3300 1900 50  0000 C CNN
 F 2 "" H 3200 2000 50  0000 C CNN
@@
 $EndComp
 $Comp
-L CONN_01X03 P?
+L CONN_01X03 P8
 U 1 1 583A60A2
 P 2900 2000
-F 0 "P?" H 2900 1800 50  0000 C CNN
+F 0 "P8" H 2900 1800 50  0000 C CNN
 F 1 "CONN_01X03" V 3000 1900 50  0000 C CNN
 F 2 "" H 2900 2000 50  0000 C CNN
@@
 $EndComp
 $Comp
-L CONN_01X04 P?
+L CONN_01X04 P14
 U 1 1 583A6112
 P 5250 2150
-F 0 "P?" H 5250 2400 50  0000 C CNN
+F 0 "P14" H 5250 2400 50  0000 C CNN
 F 1 "CONN_01X04" V 5350 2150 50  0000 C CNN
 F 2 "" H 5250 2150 50  0000 C CNN
@@
 Wire Wire Line
 	4650 2400 4650 2650
-Connection ~ 4900 2500
-$Comp
-L GND #PWR04
+$Comp
+L GND #PWR014
 U 1 1 583A6463
 P 4900 2650
-F 0 "#PWR04" H 4900 2400 50  0001 C CNN
+F 0 "#PWR014" H 4900 2400 50  0001 C CNN
 F 1 "GND" H 4900 2500 50  0000 C CNN
 F 2 "" H 4900 2650 50  0000 C CNN
@@
 $EndComp
 $Comp
-L +5V #PWR05
-U 1 1 583A64AD
-P 4650 2650
-F 0 "#PWR05" H 4650 2500 50  0001 C CNN
-F 1 "+5V" H 4650 2790 50  0000 C CNN
-F 2 "" H 4650 2650 50  0000 C CNN
-F 3 "" H 4650 2650 50  0000 C CNN
-	1    4650 2650
-	-1   0    0    1
-$EndComp
-$Comp
-L CONN_01X03 P?
+L CONN_01X03 P12
 U 1 1 583A6DC1
 P 3200 3500
-F 0 "P?" H 3200 3300 50  0000 C CNN
+F 0 "P12" H 3200 3300 50  0000 C CNN
 F 1 "CONN_01X03" V 3300 3400 50  0000 C CNN
 F 2 "" H 3200 3500 50  0000 C CNN
@@
 $EndComp
 $Comp
-L CONN_01X03 P?
+L CONN_01X03 P9
 U 1 1 583A6DC7
 P 2900 3500
-F 0 "P?" H 2900 3300 50  0000 C CNN
+F 0 "P9" H 2900 3300 50  0000 C CNN
 F 1 "CONN_01X03" V 3000 3400 50  0000 C CNN
 F 2 "" H 2900 3500 50  0000 C CNN
@@
 $EndComp
 $Comp
-L CONN_01X03 P?
+L CONN_01X03 P13
 U 1 1 583A7499
 P 3200 5000
-F 0 "P?" H 3200 4800 50  0000 C CNN
+F 0 "P13" H 3200 4800 50  0000 C CNN
 F 1 "CONN_01X03" V 3300 4900 50  0000 C CNN
 F 2 "" H 3200 5000 50  0000 C CNN
@@
 $EndComp
 $Comp
-L CONN_01X03 P?
+L CONN_01X03 P10
 U 1 1 583A749F
 P 2900 5000
-F 0 "P?" H 2900 4800 50  0000 C CNN
+F 0 "P10" H 2900 4800 50  0000 C CNN
 F 1 "CONN_01X03" V 3000 4900 50  0000 C CNN
 F 2 "" H 2900 5000 50  0000 C CNN
@@
 ENABLE
 $Comp
-L CONN_01X04 P?
+L CONN_01X04 P15
 U 1 1 583AB31E
 P 5250 3650
-F 0 "P?" H 5250 3900 50  0000 C CNN
+F 0 "P15" H 5250 3900 50  0000 C CNN
 F 1 "CONN_01X04" V 5350 3650 50  0000 C CNN
 F 2 "" H 5250 3650 50  0000 C CNN
@@
 $EndComp
 $Comp
-L CONN_01X04 P?
+L CONN_01X04 P16
 U 1 1 583AB453
 P 5250 5150
-F 0 "P?" H 5250 5400 50  0000 C CNN
+F 0 "P16" H 5250 5400 50  0000 C CNN
 F 1 "CONN_01X04" V 5350 5150 50  0000 C CNN
 F 2 "" H 5250 5150 50  0000 C CNN
@@
 Wire Wire Line
 	5050 3800 4550 3800
-Connection ~ 4900 4000
 Wire Wire Line
 	4550 3900 4650 3900
 Wire Wire Line
 	4650 3900 4650 4150
-Connection ~ 4900 5500
 Wire Wire Line
 	4550 5400 4650 5400
@@
 	4650 5400 4650 5650
 $Comp
-L +5V #PWR06
-U 1 1 583AC633
-P 4650 4150
-F 0 "#PWR06" H 4650 4000 50  0001 C CNN
-F 1 "+5V" H 4650 4290 50  0000 C CNN
-F 2 "" H 4650 4150 50  0000 C CNN
-F 3 "" H 4650 4150 50  0000 C CNN
-	1    4650 4150
-	-1   0    0    1
-$EndComp
-$Comp
-L +5V #PWR07
-U 1 1 583AC686
-P 4650 5650
-F 0 "#PWR07" H 4650 5500 50  0001 C CNN
-F 1 "+5V" H 4650 5790 50  0000 C CNN
-F 2 "" H 4650 5650 50  0000 C CNN
-F 3 "" H 4650 5650 50  0000 C CNN
-	1    4650 5650
-	-1   0    0    1
-$EndComp
-$Comp
-L GND #PWR08
+L GND #PWR015
 U 1 1 583AC781
 P 4900 4150
-F 0 "#PWR08" H 4900 3900 50  0001 C CNN
+F 0 "#PWR015" H 4900 3900 50  0001 C CNN
 F 1 "GND" H 4900 4000 50  0000 C CNN
 F 2 "" H 4900 4150 50  0000 C CNN
@@
 $EndComp
 $Comp
-L GND #PWR09
+L GND #PWR016
 U 1 1 583AC894
 P 4900 5650
-F 0 "#PWR09" H 4900 5400 50  0001 C CNN
+F 0 "#PWR016" H 4900 5400 50  0001 C CNN
 F 1 "GND" H 4900 5500 50  0000 C CNN
 F 2 "" H 4900 5650 50  0000 C CNN
@@
 $EndComp
 $Comp
-L CONN_01X02 P?
-U 1 1 583AD129
-P 6250 1350
-F 0 "P?" H 6250 1500 50  0000 C CNN
-F 1 "CONN_01X02" V 6350 1350 50  0000 C CNN
-F 2 "" H 6250 1350 50  0000 C CNN
-F 3 "" H 6250 1350 50  0000 C CNN
-	1    6250 1350
-	0    -1   -1   0
-$EndComp
-$Comp
-L CP C?
+L CP C3
 U 1 1 583AD1F5
 P 5700 2150
-F 0 "C?" H 5725 2250 50  0000 L CNN
+F 0 "C3" H 5725 2250 50  0000 L CNN
 F 1 "CP" H 5725 2050 50  0000 L CNN
 F 2 "" H 5738 2000 50  0000 C CNN
@@
 $EndComp
 Wire Wire Line
-	4550 1800 6200 1800
+	4550 1800 6700 1800
 Wire Wire Line
 	5700 1800 5700 2000
 Wire Wire Line
-	5700 2500 5700 2300
-$Comp
-L CP C?
+	5700 2300 5700 2650
+$Comp
+L CP C4
 U 1 1 583AD810
 P 5700 3600
-F 0 "C?" H 5725 3700 50  0000 L CNN
+F 0 "C4" H 5725 3700 50  0000 L CNN
 F 1 "CP" H 5725 3500 50  0000 L CNN
 F 2 "" H 5738 3450 50  0000 C CNN
@@
 $EndComp
 $Comp
-L CP C?
+L CP C5
 U 1 1 583AD8AF
 P 5700 5150
-F 0 "C?" H 5725 5250 50  0000 L CNN
+F 0 "C5" H 5725 5250 50  0000 L CNN
 F 1 "CP" H 5725 5050 50  0000 L CNN
 F 2 "" H 5738 5000 50  0000 C CNN
@@
 	5700 3300 5700 3450
 Wire Wire Line
-	5700 4000 5700 3750
+	5700 3750 5700 4150
 Wire Wire Line
 	6200 4800 4550 4800
@@
 	5700 4800 5700 5000
 Wire Wire Line
-	5700 5500 5700 5300
+	5700 5300 5700 5650
 Connection ~ 5700 1800
-Wire Wire Line
-	6200 1550 6200 4800
 Connection ~ 5700 3300
 Connection ~ 5700 4800
-Connection ~ 6200 3300
-Connection ~ 6200 1800
-Wire Wire Line
-	6300 5500 6300 1550
-Connection ~ 5700 5500
-$Comp
-L +5V #PWR?
+$Comp
+L +5V #PWR017
 U 1 1 583B0DD4
 P 2400 2150
-F 0 "#PWR?" H 2400 2000 50  0001 C CNN
+F 0 "#PWR017" H 2400 2000 50  0001 C CNN
 F 1 "+5V" H 2400 2290 50  0000 C CNN
 F 2 "" H 2400 2150 50  0000 C CNN
@@
 Connection ~ 2400 2100
 $Comp
-L +5V #PWR?
+L +5V #PWR018
 U 1 1 583B180A
 P 2400 3650
-F 0 "#PWR?" H 2400 3500 50  0001 C CNN
+F 0 "#PWR018" H 2400 3500 50  0001 C CNN
 F 1 "+5V" H 2400 3790 50  0000 C CNN
 F 2 "" H 2400 3650 50  0000 C CNN
@@
 $EndComp
 $Comp
-L +5V #PWR?
+L +5V #PWR019
 U 1 1 583B1885
 P 2400 5150
-F 0 "#PWR?" H 2400 5000 50  0001 C CNN
+F 0 "#PWR019" H 2400 5000 50  0001 C CNN
 F 1 "+5V" H 2400 5290 50  0000 C CNN
 F 2 "" H 2400 5150 50  0000 C CNN
@@
 	2700 5100 2400 5100
 Connection ~ 2400 5100
+$Comp
+L GND #PWR020
+U 1 1 5840D9F7
+P 5700 2650
+F 0 "#PWR020" H 5700 2400 50  0001 C CNN
+F 1 "GND" H 5700 2500 50  0000 C CNN
+F 2 "" H 5700 2650 50  0000 C CNN
+F 3 "" H 5700 2650 50  0000 C CNN
+	1    5700 2650
+	1    0    0    -1
+$EndComp
+$Comp
+L GND #PWR021
+U 1 1 5840DB54
+P 5700 4150
+F 0 "#PWR021" H 5700 3900 50  0001 C CNN
+F 1 "GND" H 5700 4000 50  0000 C CNN
+F 2 "" H 5700 4150 50  0000 C CNN
+F 3 "" H 5700 4150 50  0000 C CNN
+	1    5700 4150
+	1    0    0    -1
+$EndComp
+$Comp
+L GND #PWR022
+U 1 1 5840DC8F
+P 5700 5650
+F 0 "#PWR022" H 5700 5400 50  0001 C CNN
+F 1 "GND" H 5700 5500 50  0000 C CNN
+F 2 "" H 5700 5650 50  0000 C CNN
+F 3 "" H 5700 5650 50  0000 C CNN
+	1    5700 5650
+	1    0    0    -1
+$EndComp
+Wire Wire Line
+	4550 5500 4900 5500
+Connection ~ 4900 5500
+Wire Wire Line
+	4550 4000 4900 4000
+Connection ~ 4900 4000
+Wire Wire Line
+	4550 2500 4900 2500
+Connection ~ 4900 2500
+Text GLabel 6700 1800 2    60   Input ~ 0
+EXT-V
+Wire Wire Line
+	6200 1300 6200 4800
+Connection ~ 6200 1800
+Connection ~ 6200 3300
+$Comp
+L +3.3V #PWR023
+U 1 1 58411F6E
+P 4650 2650
+F 0 "#PWR023" H 4650 2500 50  0001 C CNN
+F 1 "+3.3V" H 4650 2790 50  0000 C CNN
+F 2 "" H 4650 2650 50  0000 C CNN
+F 3 "" H 4650 2650 50  0000 C CNN
+	1    4650 2650
+	-1   0    0    1
+$EndComp
+$Comp
+L +3.3V #PWR024
+U 1 1 584125D2
+P 4650 4150
+F 0 "#PWR024" H 4650 4000 50  0001 C CNN
+F 1 "+3.3V" H 4650 4290 50  0000 C CNN
+F 2 "" H 4650 4150 50  0000 C CNN
+F 3 "" H 4650 4150 50  0000 C CNN
+	1    4650 4150
+	-1   0    0    1
+$EndComp
+$Comp
+L +3.3V #PWR025
+U 1 1 584126A0
+P 4650 5650
+F 0 "#PWR025" H 4650 5500 50  0001 C CNN
+F 1 "+3.3V" H 4650 5790 50  0000 C CNN
+F 2 "" H 4650 5650 50  0000 C CNN
+F 3 "" H 4650 5650 50  0000 C CNN
+	1    4650 5650
+	-1   0    0    1
+$EndComp
+$Comp
+L PWR_FLAG #FLG026
+U 1 1 58434718
+P 6200 1300
+F 0 "#FLG026" H 6200 1395 50  0001 C CNN
+F 1 "PWR_FLAG" H 6200 1480 50  0000 C CNN
+F 2 "" H 6200 1300 50  0000 C CNN
+F 3 "" H 6200 1300 50  0000 C CNN
+	1    6200 1300
+	1    0    0    -1
+$EndComp
 $EndSCHEMATC
